Commit message: Fix field camera FoV.

File: tmplanner_tools/sim/descriptions/firefly_base_gps_cam_field.xacro (robot description, xacro)
@@ -69,5 +69,5 @@
     frame_rate="0.2"
     camera_suffix="sim"
-    horizontal_fov="0.824"
+    horizontal_fov="1.187"
     image_format="R8G8B8"
     min_distance="0.02"
@@ -77,5 +77,5 @@
     enable_visual="true">
     <box size="0.02 0.02 0.02" />
-    <origin xyz="0 0 -0.05" rpy="0 ${pi/2} 0" />
+    <origin xyz="0.0408 0.1519 -0.0621" rpy="0 ${pi/2} 0" />
   </xacro:camera_macro>
   <xacro:if value="$(arg enable_ground_truth)">
